File: proto1/macadamia.kicad_pcb (KiCad board)
At the start: 2 copper layers, 50 x 50 mm, 12 parts, among them J1 Conn_01x05_Pin, J2 DIN-6, J3 DIN-6, Q1 AO3400A, Q2 AO3401A, Q3 AO3401A, Q4 AO3400A

Commit message: proto1: Fix pfet orientation
Parts:
- moved R4 7.22 mm to (170.0, 60.8), turned to 0 degrees
Connections:
- Q2 pad 2: /Comms Interface/MCU_RX -> +3.3V
- Q2 pad 3: +3.3V -> /Comms Interface/MCU_RX
- Q3 pad 2: /Comms Interface/COMMS -> +5V
- Q3 pad 3: +5V -> /Comms Interface/COMMS
Routing:
- net +3.3V: track 14.8 -> 7.37 mm, vias 1 -> 0
- net /Comms Interface/MCU_RX: track 14.2 -> 18.0 mm
- net /Comms Interface/MCU_RX_PU: track 13.2 -> 9.70 mm
- net +5V: track 22.9 -> 20.8 mm
- net /Comms Interface/COMMS: track 14.8 -> 16.6 mm
